File: hardware/pcb/moonlamp.brd (EAGLE design)
At the start: 96 x 96 mm, 57 parts, among them IC1 MEGA8-AI, IC2 DS1307, IC4 78L05SMD, Q2 32,768kHz, T1 IRLML2502, T10 IRLML2502, T11 IRLML2502, T12 IRLML2502, T13 IRLML2502, T2 IRLML2502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

Commit message: cleaned up schematic
Connections:
- net N$1 renamed TOUCH
- net N$15 renamed SDA
- net N$39 renamed RESET
Changed lines of the file:
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@@
 <layer number="23" name="tOrigins" color="15" fill="1" visible="yes" active="yes"/>
 <layer number="24" name="bOrigins" color="15" fill="1" visible="yes" active="yes"/>
-<layer number="25" name="tNames" color="7" fill="1" visible="yes" active="yes"/>
+<layer number="25" name="tNames" color="7" fill="1" visible="no" active="yes"/>
 <layer number="26" name="bNames" color="7" fill="1" visible="no" active="yes"/>
 <layer number="27" name="tValues" color="7" fill="1" visible="no" active="yes"/>
 <layer number="28" name="bValues" color="7" fill="1" visible="no" active="yes"/>
-<layer number="29" name="tStop" color="7" fill="3" visible="yes" active="yes"/>
-<layer number="30" name="bStop" color="7" fill="6" visible="yes" active="yes"/>
+<layer number="29" name="tStop" color="7" fill="3" visible="no" active="yes"/>
+<layer number="30" name="bStop" color="7" fill="6" visible="no" active="yes"/>
 <layer number="31" name="tCream" color="7" fill="4" visible="no" active="yes"/>
 <layer number="32" name="bCream" color="7" fill="5" visible="no" active="yes"/>
@@
 <wire x1="69.9525" y1="70.1675" x2="69.85" y2="70.27" width="0.4064" layer="1"/>
 </signal>
-<signal name="N$15">
+<signal name="SDA">
 <contactref element="IC2" pad="5"/>
-<contactref element="IC1" pad="27"/>
 <contactref element="R3" pad="1"/>
 <contactref element="SDA" pad="TP"/>
@@
 <wire x1="34.6075" y1="59.3725" x2="36.0934" y2="57.8866" width="0.4064" layer="1"/>
 <wire x1="36.0934" y1="57.8866" x2="37.7825" y2="57.8866" width="0.4064" layer="1"/>
-<wire x1="64.2874" y1="62.795" x2="59.4425" y2="62.795" width="0.4064" layer="1"/>
 <wire x1="59.4425" y1="62.795" x2="59.055" y2="63.1825" width="0.4064" layer="1"/>
 <via x="59.055" y="63.1825" extent="1-16" drill="0.3048" shape="octagon"/>
@@
 <wire x1="37.7825" y1="56.515" x2="37.7825" y2="57.8866" width="0.4064" layer="1"/>
 <wire x1="55.245" y1="59.69" x2="55.245" y2="60.96" width="0.4064" layer="1"/>
+<contactref element="IC1" pad="27"/>
+<wire x1="59.4425" y1="62.795" x2="64.2874" y2="62.795" width="0.4064" layer="1"/>
 </signal>
 <signal name="SCL">
 <contactref element="IC2" pad="6"/>
-<contactref element="IC1" pad="28"/>
 <contactref element="R2" pad="1"/>
 <contactref element="SCL" pad="TP"/>
@@
 <wire x1="38.315" y1="60.11" x2="39.0525" y2="59.3725" width="0.4064" layer="1"/>
 <wire x1="39.0525" y1="59.3725" x2="39.0525" y2="57.8866" width="0.4064" layer="1"/>
-<wire x1="64.2874" y1="61.995" x2="55.245" y2="61.995" width="0.4064" layer="1"/>
 <wire x1="55.245" y1="61.995" x2="54.375" y2="61.995" width="0.4064" layer="1"/>
 <wire x1="54.375" y1="61.995" x2="47.9425" y2="55.5625" width="0.4064" layer="1"/>
@@
 <wire x1="39.0525" y1="56.515" x2="39.0525" y2="57.8866" width="0.4064" layer="1"/>
 <wire x1="55.245" y1="63.5" x2="55.245" y2="61.995" width="0.4064" layer="1"/>
+<contactref element="IC1" pad="28"/>
+<wire x1="55.245" y1="61.995" x2="64.2874" y2="61.995" width="0.4064" layer="1"/>
 </signal>
 <signal name="N$3">
@@
 <wire x1="74.93" y1="69.85" x2="77.47" y2="72.39" width="0.4064" layer="1"/>
 <wire x1="77.47" y1="72.39" x2="77.47" y2="73.025" width="0.4064" layer="1"/>
-</signal>
-<signal name="N$39">
-<contactref element="C3" pad="2"/>
-<contactref element="R1" pad="1"/>
-<contactref element="IC1" pad="29"/>
-<contactref element="ISP" pad="1"/>
-<wire x1="64.2874" y1="61.195" x2="65.17" y2="61.195" width="0.4064" layer="1"/>
-<wire x1="65.17" y1="61.195" x2="65.7225" y2="60.6425" width="0.4064" layer="1"/>
-<via x="65.7225" y="60.6425" extent="1-16" drill="0.3048" shape="octagon"/>
-<wire x1="65.7225" y1="60.6425" x2="64.4525" y2="60.6425" width="0.4064" layer="16"/>
-<wire x1="64.4525" y1="60.6425" x2="59.69" y2="65.405" width="0.4064" layer="16"/>
-<wire x1="59.69" y1="65.405" x2="59.69" y2="68.2625" width="0.4064" layer="16"/>
-<via x="59.69" y="68.2625" extent="1-16" drill="0.3048" shape="octagon"/>
-<wire x1="59.69" y1="68.2625" x2="64.4525" y2="73.025" width="0.4064" layer="1"/>
-<wire x1="64.4525" y1="73.025" x2="68.2625" y2="73.025" width="0.4064" layer="1"/>
-<wire x1="68.2625" y1="73.025" x2="69.85" y2="73.025" width="0.4064" layer="1"/>
-<wire x1="69.85" y1="73.025" x2="72.39" y2="73.025" width="0.4064" layer="1"/>
-<wire x1="69.85" y1="71.97" x2="69.85" y2="73.025" width="0.4064" layer="1"/>
-<wire x1="68.2625" y1="71.995" x2="68.2625" y2="73.025" width="0.4064" layer="1"/>
 </signal>
 <signal name="N$10">
@@
 <wire x1="40.3225" y1="67.1445" x2="39.031" y2="68.436" width="0.4064" layer="1"/>
 </signal>
-<signal name="N$1">
+<signal name="N$2">
+<contactref element="ADC7" pad="1"/>
+<contactref element="IC1" pad="22"/>
+<wire x1="67.38" y1="65.8876" x2="67.38" y2="68.8275" width="0.4064" layer="1"/>
+<wire x1="67.38" y1="68.8275" x2="66.9925" y2="69.215" width="0.4064" layer="1"/>
+<wire x1="66.9925" y1="69.215" x2="64.77" y2="69.215" width="0.4064" layer="1"/>
+</signal>
+<signal name="N$38">
+<contactref element="IC1" pad="23"/>
+<contactref element="PC0" pad="1"/>
+<wire x1="66.58" y1="65.8876" x2="66.58" y2="67.405" width="0.4064" layer="1"/>
+<wire x1="66.58" y1="67.405" x2="66.3575" y2="67.6275" width="0.4064" layer="1"/>
+<wire x1="66.3575" y1="67.6275" x2="64.77" y2="67.6275" width="0.4064" layer="1"/>
+</signal>
+<signal name="RESET">
+<contactref element="ISP" pad="1"/>
+<contactref element="C3" pad="2"/>
+<contactref element="R1" pad="1"/>
+<contactref element="IC1" pad="29"/>
+<wire x1="64.2874" y1="61.195" x2="65.17" y2="61.195" width="0.4064" layer="1"/>
+<wire x1="65.17" y1="61.195" x2="65.7225" y2="60.6425" width="0.4064" layer="1"/>
+<via x="65.7225" y="60.6425" extent="1-16" drill="0.3048" shape="octagon"/>
+<wire x1="65.7225" y1="60.6425" x2="64.4525" y2="60.6425" width="0.4064" layer="16"/>
+<wire x1="64.4525" y1="60.6425" x2="59.69" y2="65.405" width="0.4064" layer="16"/>
+<wire x1="59.69" y1="65.405" x2="59.69" y2="68.2625" width="0.4064" layer="16"/>
+<via x="59.69" y="68.2625" extent="1-16" drill="0.3048" shape="octagon"/>
+<wire x1="59.69" y1="68.2625" x2="64.4525" y2="73.025" width="0.4064" layer="1"/>
+<wire x1="64.4525" y1="73.025" x2="68.2625" y2="73.025" width="0.4064" layer="1"/>
+<wire x1="68.2625" y1="73.025" x2="69.85" y2="73.025" width="0.4064" layer="1"/>
+<wire x1="69.85" y1="71.97" x2="69.85" y2="73.025" width="0.4064" layer="1"/>
+<wire x1="68.2625" y1="71.995" x2="68.2625" y2="73.025" width="0.4064" layer="1"/>
+<wire x1="69.85" y1="73.025" x2="72.39" y2="73.025" width="0.4064" layer="1"/>
+</signal>
+<signal name="TOUCH">
 <contactref element="IC1" pad="12"/>
 <contactref element="R4" pad="2"/>
 <contactref element="C2" pad="2"/>
 <contactref element="TOUCH" pad="1"/>
-<wire x1="72.8726" y1="61.195" x2="80.41" y2="61.195" width="0.4064" layer="1"/>
 <wire x1="80.41" y1="61.195" x2="80.645" y2="60.96" width="0.4064" layer="1"/>
 <wire x1="80.645" y1="60.96" x2="80.645" y2="59.905" width="0.4064" layer="1"/>
@@
 <wire x1="80.645" y1="64.135" x2="80.645" y2="60.96" width="0.4064" layer="16"/>
 <via x="80.645" y="60.96" extent="1-16" drill="0.3048" shape="octagon"/>
-</signal>
-<signal name="N$2">
-<contactref element="ADC7" pad="1"/>
-<contactref element="IC1" pad="22"/>
-<wire x1="67.38" y1="65.8876" x2="67.38" y2="68.8275" width="0.4064" layer="1"/>
-<wire x1="67.38" y1="68.8275" x2="66.9925" y2="69.215" width="0.4064" layer="1"/>
-<wire x1="66.9925" y1="69.215" x2="64.77" y2="69.215" width="0.4064" layer="1"/>
-</signal>
-<signal name="N$38">
-<contactref element="IC1" pad="23"/>
-<contactref element="PC0" pad="1"/>
-<wire x1="66.58" y1="65.8876" x2="66.58" y2="67.405" width="0.4064" layer="1"/>
-<wire x1="66.58" y1="67.405" x2="66.3575" y2="67.6275" width="0.4064" layer="1"/>
-<wire x1="66.3575" y1="67.6275" x2="64.77" y2="67.6275" width="0.4064" layer="1"/>
+<wire x1="80.41" y1="61.195" x2="72.8726" y2="61.195" width="0.4064" layer="1"/>
 </signal>
 </signals>
