File: hardware/pcb/moonlamp.sch (EAGLE design)
At the start: 57 parts, among them IC1 MEGA8-AI, IC2 DS1307, IC4 78L05SMD, Q2 32,768kHz, T1 IRLML2502, T10 IRLML2502, T11 IRLML2502, T12 IRLML2502, T13 IRLML2502, T2 IRLML2502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

Commit message: cleaned up schematic
Connections:
- net N$1 renamed TOUCH
- net N$15 renamed SDA
- net N$39 renamed RESET
Other:
- note added: "LED drivers + moon layout"
- note added: "microcontroller + ISP"
- note added: "real time clock"
- note added: "touch-pin (capacity based)"
- note added: "voltage controller"
- moved on the sheet: +, -, 5V, ADC7, B1, C1, C15, C2, C3, C4, C5, C6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
